Commit message: feat(phase3): cooperative fleet map, the fleet frame, and selective updates
Two robots, two SLAM maps, one composited map that BOTH global costmaps plan in.
Phases 3 and 4 merged per docs/DELIVERY_PLAN_COMPRESSED.md; the ramp A/B moves to
Session B by decision, and what ships here instead is the ramp filter plumbing,
wired and measured contributing exactly nothing.

Bringup split so one launch can run one robot and another the whole fleet without
either including the other: amr_gazebo.spawn.world_actions owns the world
singletons, robot_stack.launch.py owns one robot's stack, fleet_nav.launch.py loops
over fleet.yaml. amr1_nav.launch.py stays strictly single-robot - three Phase 1/2
evidence launches include it by name, and making it a fleet launch would have
silently doubled the graph load under every recorded measurement.

FleetMapNode publishes its static frames and a fixed-extent map in its constructor.
Both are load-bearing: Costmap2DROS blocks on the transform during activation with
no timeout on the lifecycle manager's side, and it defaults to a 5x5 m window at the
origin while both robots spawn outside it.

Selective updates are scored - frontier, occupancy change, recency, revisit penalty -
under an invariant the weights must satisfy: no positive term may be vetoed by the
revisit penalty. The first weights violated it and deferred a new obstacle on a
much-travelled corridor, which is the exact failure a visit-count-only policy has.
A test asserts the invariant directly.

Measured:
  dual bringup    53 nodes, both stacks active, no collisions
  fleet map       680x400 @ 0.05 m, RELIABLE/TRANSIENT_LOCAL, matched by both
                  global costmaps; static TFs at (-11, -/+1.5, 0)
  selective       41 candidates, 23 accepted, 18 deferred (43.9 %)
  concurrent      both SUCCEEDED, 18.8 s / 11.3 s, closest approach 3.000 m
  ramp filter     loaded and active, min cost 0 over 272k known cells while
                  ~24k cells are costed
  recovery A/B    suppressed: one 56.69 s halt, 0 recoveries, allowance 1e6
                  control:    8 halts capped at ~10 s, 6x "Failed to make
                              progress", 2 recoveries DURING a halt
  regression      Phase 1 baseline unchanged except replan count 5 -> 1, which
                  is a consequence of the static layer now reading a
                  rate-limited fleet map rather than slam_toolbox directly

The recovery A/B is the Phase 2 carry-over. Phase 2 could only show the mechanism
operates; its longest halt was 0.80 s against a 10 s allowance. A barrier that never
moves produces a halt that does not end, and the control arm shows Nav2 declaring the
robot stuck while the safety gate is deliberately holding it.

Two environment findings, both silent:
  - two Nav2 stacks exceed CycloneDDS's default MaxAutoParticipantIndex of 9, and
    the resulting node-creation failures land on whichever servers start last,
    reading as "the second robot is broken" rather than a host-wide limit
  - this environment already exports CYCLONEDDS_URI, so the natural ${VAR:-default}
    fix is a no-op and plain assignment would drop the existing interface pinning;
    ws.sh appends, because CycloneDDS merges a comma-separated list

Also corrected, found by running the regression rather than reading it: /plan moved
to the fleet frame, and nav_goal_run was still applying the spawn offset on top -
writing a route that starts at (-22.00, -3.00) where the robot starts at
(-11.00, -1.50), while every derived metric stayed correct because they are all
translation-invariant.

colcon build 9 packages / 0 errors, pytest 171 passed, flake8 + black clean.

File: src/amr_gazebo/worlds/warehouse.sdf.xacro (robot description, xacro)
@@ -25,4 +25,19 @@
        from the effect being measured, so actors can be switched off. -->
   <xacro:arg name="with_actors" default="true"/>
+  <!-- An immovable barrier parked across the aisle, defaulted OFF so every run
+       recorded before Phase 3 still describes the world it was measured in.
+       Phase 2's recovery-suppression A/B could only show that the mechanism
+       OPERATES, never that it was NEEDED: the longest halt it produced was 0.80 s
+       against a 10 s movement_time_allowance, because a walking pedestrian clears
+       the sector in under a second. A barrier that never moves produces a halt that
+       does not end, which is the condition the suppression exists for. -->
+  <xacro:arg name="with_static_obstacle" default="false"/>
+  <xacro:arg name="obstacle_x" default="-5.0"/>
+  <xacro:arg name="obstacle_y" default="0.0"/>
+  <!-- Spans the full 5.5 m aisle by default. A gap the robot could plan through
+       would let Nav2 route around it, and the halt would end as soon as it did. -->
+  <xacro:arg name="obstacle_size_y" default="5.5"/>
+  <xacro:arg name="obstacle_size_x" default="0.40"/>
+  <xacro:arg name="obstacle_size_z" default="1.20"/>
   <xacro:property name="ramp_angle_deg" value="$(arg ramp_angle_deg)"/>
   <xacro:property name="ramp_angle" value="${radians(ramp_angle_deg)}"/>
@@ -207,4 +222,31 @@
     <xacro:rack_row side="north" y="${rack_row_y}"/>
     <xacro:rack_row side="south" y="${-rack_row_y}"/>
+    <!-- ==================== Static barrier (optional) ====================
+         Ordinary static geometry, emitted in the same shape as a rack. Because it
+         is a <model> with a <collision><geometry><box>, world_geometry.static_boxes
+         picks it up for free, so the LiDAR-only dynamic/static classifier in
+         nav_goal_run scores it as static with no code change. -->
+    <xacro:if value="${'$(arg with_static_obstacle)'.lower() == 'true'}">
+    <model name="static_barrier">
+      <static>true</static>
+      <pose>$(arg obstacle_x) $(arg obstacle_y) ${$(arg obstacle_size_z) / 2.0} 0 0 0</pose>
+      <link name="link">
+        <collision name="collision">
+          <geometry>
+            <box><size>$(arg obstacle_size_x) $(arg obstacle_size_y) $(arg obstacle_size_z)</size></box>
+          </geometry>
+        </collision>
+        <visual name="visual">
+          <geometry>
+            <box><size>$(arg obstacle_size_x) $(arg obstacle_size_y) $(arg obstacle_size_z)</size></box>
+          </geometry>
+          <material>
+            <ambient>0.65 0.15 0.10 1</ambient>
+            <diffuse>0.85 0.20 0.15 1</diffuse>
+          </material>
+        </visual>
+      </link>
+    </model>
+    </xacro:if>
     <!-- ==================== Moving obstacles ====================
          Confirmed in smoke test 1: visible to the LiDAR, reaching the Nav2

Commit message: feat(phase7): TrafficControlNode — the yield protocol and its escalation path
The last requirement with no implementation. Phase 6 shipped the local half of
assignment 3.2 (FleetTrajectoryLayer) and left the escalation half with plumbing
only: a priority-150 cmd_vel_yield mux channel, timeout-based release, and a
unit-tested conflict predicate with no caller.

TrafficControlNode is central ONLY for escalation (docs/ENGINEERING_NOTES.md rule 7). It refuses
to act while the predicted closest approach is still opening, so a conflict the
local layer is resolving is left to it, and every conflict it declines is counted
beside every one it takes — that ordering is what the evidence has to show.

Arbitration constants are derived from fleet.yaml, not tuned:
  priority        gross mass, ties on declaration order -> amr1 90 kg > amr2 23 kg
  conflict radius 1.94 m = r(amr1) + r(amr2) + d_safe(amr1 @ cruise)
No robot is named in the arbiter; the assignment's "AMR-2 yields to AMR-1" falls
out of the mass column, and the tests assert that changing the masses changes the
yield direction.

Evidence — one forced narrow-intersection conflict (results/phase7_yield.*):
the Phase 3 barrier split around a 3.0 m gap, both goals beyond it, amr2's
dispatch held back 5 s so both reach the gap together. Two escalations, amr2
yields both times, held 1.0 s and 15.2 s, both released on "conflict cleared",
0 recovery behaviours during either hold, movement_time_allowance read back at
1e6 on entry and 10 s after release, SafetyGate blocking on 0 of 326 held cycles
so the stop is the arbiter's and nothing else's. Both goals SUCCEEDED.

The 15.2 s hold outlasts the 10 s allowance, which is the condition Phase 3
measured recoveries firing under — but the control arm of THIS run has not been
executed, so necessity still rests on Phase 3's A/B and the log says so.

Also: obstacle_gap_y splits the static barrier (0.0 keeps the solid wall every
earlier run was measured against), fleet_mission gains dispatch_offsets (all-zero
default preserves Phase 3's simultaneous dispatch), and with_traffic_control
defaults on but is skipped where there is no mux to command through.

9 packages / 0 errors, pytest 241 passed (223 + 18 new), flake8 + black clean.

File: src/amr_gazebo/worlds/warehouse.sdf.xacro (robot description, xacro)
@@ -38,4 +38,13 @@
        would let Nav2 route around it, and the halt would end as soon as it did. -->
   <xacro:arg name="obstacle_size_y" default="5.5"/>
+  <!-- Width of a gap left in the MIDDLE of that barrier, turning it from a wall
+       into a constriction. 0 keeps the solid wall every run before Phase 7 was
+       measured against. A gap makes both robots' global plans converge on the
+       same few metres of aisle, which is what a narrow intersection IS: not a
+       place they might collide, but the only place either can pass. Sized in
+       Phase 7 so that a robot centred in the gap still clears the barrier ends
+       by more than its own braking envelope - a gap the SafetyGate halts inside
+       would measure the gate, not the yield protocol. -->
+  <xacro:arg name="obstacle_gap_y" default="0.0"/>
   <xacro:arg name="obstacle_size_x" default="0.40"/>
   <xacro:arg name="obstacle_size_z" default="1.20"/>
@@ -227,25 +236,43 @@
          picks it up for free, so the LiDAR-only dynamic/static classifier in
          nav_goal_run scores it as static with no code change. -->
+    <xacro:macro name="barrier_segment" params="name y len">
+      <model name="${name}">
+        <static>true</static>
+        <pose>$(arg obstacle_x) ${y} ${$(arg obstacle_size_z) / 2.0} 0 0 0</pose>
+        <link name="link">
+          <collision name="collision">
+            <geometry>
+              <box><size>$(arg obstacle_size_x) ${len} $(arg obstacle_size_z)</size></box>
+            </geometry>
+          </collision>
+          <visual name="visual">
+            <geometry>
+              <box><size>$(arg obstacle_size_x) ${len} $(arg obstacle_size_z)</size></box>
+            </geometry>
+            <material>
+              <ambient>0.65 0.15 0.10 1</ambient>
+              <diffuse>0.85 0.20 0.15 1</diffuse>
+            </material>
+          </visual>
+        </link>
+      </model>
+    </xacro:macro>
     <xacro:if value="${'$(arg with_static_obstacle)'.lower() == 'true'}">
-    <model name="static_barrier">
-      <static>true</static>
-      <pose>$(arg obstacle_x) $(arg obstacle_y) ${$(arg obstacle_size_z) / 2.0} 0 0 0</pose>
-      <link name="link">
-        <collision name="collision">
-          <geometry>
-            <box><size>$(arg obstacle_size_x) $(arg obstacle_size_y) $(arg obstacle_size_z)</size></box>
-          </geometry>
-        </collision>
-        <visual name="visual">
-          <geometry>
-            <box><size>$(arg obstacle_size_x) $(arg obstacle_size_y) $(arg obstacle_size_z)</size></box>
-          </geometry>
-          <material>
-            <ambient>0.65 0.15 0.10 1</ambient>
-            <diffuse>0.85 0.20 0.15 1</diffuse>
-          </material>
-        </visual>
-      </link>
-    </model>
+      <!-- One wall, or two segments with a gap between them. The segment length
+           follows from the span and the gap, so the barrier always occupies the
+           same total width and only its middle changes. -->
+      <xacro:property name="gap" value="${$(arg obstacle_gap_y)}"/>
+      <xacro:property name="span" value="${$(arg obstacle_size_y)}"/>
+      <xacro:property name="mid" value="${$(arg obstacle_y)}"/>
+      <xacro:unless value="${gap > 0.0}">
+        <xacro:barrier_segment name="static_barrier" y="${mid}" len="${span}"/>
+      </xacro:unless>
+      <xacro:if value="${gap > 0.0}">
+        <xacro:property name="seg" value="${(span - gap) / 2.0}"/>
+        <xacro:barrier_segment name="static_barrier_north"
+                               y="${mid + gap / 2.0 + seg / 2.0}" len="${seg}"/>
+        <xacro:barrier_segment name="static_barrier_south"
+                               y="${mid - gap / 2.0 - seg / 2.0}" len="${seg}"/>
+      </xacro:if>
     </xacro:if>
     <!-- ==================== Moving obstacles ====================
