Commit message: fix(phase1): correct two Phase 0 geometry defects found while planning
Both were invisible to Phase 0's own verification and both would have
corrupted Phase 1 from the first run.

1. BOTH ROBOTS SPAWNED INSIDE RACKS

   fleet.yaml placed amr1 at (-8.0, -3.0) and amr2 at (-8.0, 3.0). Rack
   rows occupy y in [2.75, 3.65] at x = -12, -8.4, -4.8, -1.2, +2.4, so
   amr1's entire 0.70 x 0.45 footprint was inside rack_south_1.

   Phase 0 missed it because both smoke tests override the spawn pose,
   and the fleet-launch check confirmed topics and TF without ever asking
   whether the robot was in free space. Robots moved into the aisle, and
   tests/test_spawn_poses_are_clear.py now renders the world, extracts
   the real obstacle geometry and asserts no footprint overlaps it. The
   guard was confirmed to fail on the original poses before being kept.

2. THE FRAME ORIGIN WAS NOT THE ROTATION CENTRE

   A differential drive pivots about its wheel axle, and Gazebo's
   DiffDrive integrates wheel encoders alone - gz::math::DiffDriveOdometry
   takes only wheel separation and radii - so the pose it publishes IS the
   axle midpoint, labelled base_footprint. The wheels sat 0.14 m aft of
   base_footprint, so odometry and TF described two different points.

   Pure translation hides this: a constant frame offset cancels, which is
   why smoke test 2 measured -0.000 m over a straight ramp traverse and
   saw nothing. Rotation exposes it. Measured, commanding a pure in-place
   turn:

       wheel odometry displacement      0.0000 m
       ground-truth displacement        0.2428 m
       disagreement                     0.2428 m   (tolerance 0.02 m)

   The laser would have swept a 0.43 m arc while TF believed 0.29 m,
   smearing the map on every turn. base_link/base_footprint moved onto
   the axle and the body offset forward instead; the robot's shape and
   weight distribution are unchanged. Re-measured: 0.0385 m peak, of
   which only 0.0193 m is an apparent offset - inside tolerance.

   That residual is physical, not modelling error, and the two runs prove
   it: the effective pivot sat ~0.019 m forward of the geometric axle
   both times (0.1214 against a true 0.14, then 0.0193 against a true
   0.0). A frictionless caster shifts the pivot forward by a constant no
   frame choice can remove. Sub-cell against 0.05 m map resolution.

   Consequence carried into Nav2: the footprint is now ASYMMETRIC about
   the origin, x in [-0.21, +0.49] for amr1. fleet_config gained
   body_x_offset/laser_x_offset/footprint_polygon so this geometry is
   derived in exactly one place - a stale copy of the laser offset was
   precisely the drift this change would otherwise have introduced.

Both smoke tests re-run against the new geometry and still pass; smoke
test 1's control-box agreement improved to -0.05 m (from -0.07 m),
independently confirming the new laser offset.

Verification: 9 packages build, 14 tests pass, flake8 + black clean.

File: src/amr_description/urdf/amr.urdf.xacro (robot description, xacro)
@@ -78,6 +78,22 @@
        on an 8 degree ramp. Adding a rear caster cured the rocking by making the base
        a rigid four-point body - which then could not pitch at all, and jammed solid
-       against the ramp toe while its wheels kept turning. -->
-  <xacro:property name="wheel_x" value="${-0.20 * base_length}"/>
+       against the ramp toe while its wheels kept turning.
+       THE FRAME ORIGIN IS THE DRIVE AXLE, NOT THE CHASSIS CENTRE.
+       A differential drive rotates about the midpoint of its wheel axle, and Gazebo's
+       DiffDrive derives odometry from wheel encoders alone, so the pose it integrates
+       IS the axle midpoint - it then labels that pose base_footprint. If base_footprint
+       were anywhere else, odometry and TF would describe two different points.
+       Phase 1 measured what that costs: commanding a pure in-place rotation, wheel
+       odometry reported 0.0000 m of displacement while Gazebo ground truth showed the
+       robot frame sweeping 0.2428 m - a 0.24 m disagreement, against a 0.02 m
+       tolerance. Sensors would have rotated about the wrong centre and smeared the map
+       on every turn. See results/odom_rotation_check.md.
+       So the wheels define the origin and the BODY is offset forward instead. The
+       robot's physical shape and its stable weight distribution are unchanged; only
+       which point is called base_link moves. One consequence is deliberate and must be
+       carried into Nav2: the footprint is now ASYMMETRIC about the origin, spanning
+       x in [-0.21, +0.49] for amr1 rather than [-0.35, +0.35]. That asymmetry is the
+       truth about how this robot sweeps when it turns. -->
+  <xacro:property name="body_x" value="${0.20 * base_length}"/>
   <xacro:property name="wheel_mass" value="${0.04 * total_mass}"/>
   <xacro:property name="body_mass" value="${total_mass - 2.0 * wheel_mass}"/>
@@ -91,5 +107,5 @@
   <link name="${prefix}base_link">
     <visual>
-      <origin xyz="0 0 ${base_height / 2.0}" rpy="0 0 0"/>
+      <origin xyz="${body_x} 0 ${base_height / 2.0}" rpy="0 0 0"/>
       <geometry>
         <box size="${base_length} ${base_width} ${base_height}"/>
@@ -100,5 +116,5 @@
     </visual>
     <collision>
-      <origin xyz="0 0 ${base_height / 2.0}" rpy="0 0 0"/>
+      <origin xyz="${body_x} 0 ${base_height / 2.0}" rpy="0 0 0"/>
       <geometry>
         <box size="${base_length} ${base_width} ${base_height}"/>
@@ -106,5 +122,5 @@
     </collision>
     <inertial>
-      <origin xyz="0 0 ${base_height / 2.0}" rpy="0 0 0"/>
+      <origin xyz="${body_x} 0 ${base_height / 2.0}" rpy="0 0 0"/>
       <mass value="${body_mass}"/>
       <!-- Solid-box inertia about the box centre. -->
@@ -151,5 +167,5 @@
       <parent link="${prefix}base_link"/>
       <child link="${prefix}${side}_wheel_link"/>
-      <origin xyz="${wheel_x} ${reflect * wheel_separation / 2.0} 0" rpy="0 0 0"/>
+      <origin xyz="0 ${reflect * wheel_separation / 2.0} 0" rpy="0 0 0"/>
       <axis xyz="0 1 0"/>
     </joint>
@@ -158,5 +174,5 @@
   <xacro:drive_wheel side="right" reflect="-1"/>
   <!-- Single passive front caster, kept low-friction so it does not fight the
-       differential drive. See the wheel_x note above for why there is exactly one. -->
+       differential drive. See the body_x note above for why there is exactly one. -->
   <xacro:macro name="caster" params="side reflect">
     <link name="${prefix}${side}_caster_link">
@@ -188,5 +204,5 @@
       <child link="${prefix}${side}_caster_link"/>
       <origin
-        xyz="${reflect * (base_length / 2.0 - caster_radius)} 0
+        xyz="${body_x + reflect * (base_length / 2.0 - caster_radius)} 0
              ${caster_radius - wheel_radius}"
         rpy="0 0 0"/>
@@ -212,5 +228,5 @@
     <parent link="${prefix}base_link"/>
     <child link="${prefix}laser"/>
-    <origin xyz="${base_length / 2.0 - 0.06} 0 ${lidar_z_in_base}" rpy="0 0 0"/>
+    <origin xyz="${body_x + base_length / 2.0 - 0.06} 0 ${lidar_z_in_base}" rpy="0 0 0"/>
   </joint>
   <link name="${prefix}imu_link">
@@ -223,5 +239,5 @@
     <parent link="${prefix}base_link"/>
     <child link="${prefix}imu_link"/>
-    <origin xyz="0 0 ${base_height / 2.0}" rpy="0 0 0"/>
+    <origin xyz="${body_x} 0 ${base_height / 2.0}" rpy="0 0 0"/>
   </joint>
   <!-- Gazebo sensors, materials and the differential drive system. -->

Commit message: feat(phase1): map artifact, goal-to-goal run, dynamic-obstacle clearance
Completes Phase 1. Exit conditions 3, 4 and 5, each with a committed
artifact and a one-command way to reproduce it:

    ros2 launch amr_bringup phase1_survey.launch.py
    ros2 launch amr_bringup phase1_nav_run.launch.py tag:=baseline \
        with_actors:=false
    ros2 launch amr_bringup phase1_nav_run.launch.py tag:=actors

EXIT 3 - SLAM MAP. Two laps of the aisle, 63.6 m. Main aisle 98.9 %
  known; rack backs and the upper plateau 0 %, because the robot never
  drove there. Occupied cells sit a median 0.000 m from the true surface,
  99.9 % within 0.15 m. The ramp is deliberately not driven: mapping while
  pitched writes the phantom ground return in as a wall, and the map shows
  exactly that wall at x = 4.9 m - the toe plus h/tan(theta), the number
  smoke test 2 measures independently.

EXIT 4 - GOAL TO GOAL. (-11.0,-1.5) -> (-0.5,+1.5), SUCCEEDED both with
  and without pedestrians: 20.5 s / 27.8 s, 11.01 m / 11.52 m executed
  against an 11.16 m plan, 5 / 4 replans, 0 / 1 recoveries. Replan count
  is routes that actually changed, not plan messages - the tree recomputes
  at 0.85 Hz regardless, so counting messages measures the tree.

EXIT 5 - DYNAMIC CLEARANCE. Head-on encounter with the aisle pedestrian,
  timed by reconstructing its trajectory from the world file. Minimum
  clearance to a dynamic obstacle 0.050 m; the robot stopped twice and
  arced around it, costing +0.51 m and +7.3 s. That 0.050 m is the floor
  of the instrument, not the gap - the actor reaches the vehicle skin
  because Gazebo actors have no collision and never yield. Reported as
  clearance, not as a collision check.

FIVE DEFECTS, THREE OF THEM FOUND BY RUNNING THE THING

  1. slam_toolbox publishes its map on the ABSOLUTE /map, escaping the
     namespace. Silent until something consumes the map; Phase 3 would
     have had two robots overwriting one global map with no error.
  2. The LiDAR was mounted inside the chassis and saw its own wheels. The
     scan plane at 0.20 m lay exactly on the wheel tops (2 * wheel_radius):
     18 beams per scan at 0.44-0.49 m off the robot itself, mapped as
     static obstacles at the robot's own position, inflated into a lethal
     blob around the start cell. The global planner failed EVERY attempt
     before the robot had moved. Sensor now on a mast at 0.35 m; 0
     self-hits in 206 scans, real returns unchanged. Both smoke tests
     re-measured at the new height and their reports regenerated.
  3. slam_toolbox's map publication is subscriber-gated, so with Nav2
     absent the survey's map saver had nothing to receive. Two full drives
     produced no artifact. survey_drive now holds a subscription open.

  Plus the two Phase 0 geometry defects fixed in 008a024, whose "why
  Phase 0 could not have caught this" is written up in the session log.

OPEN AND FLAGGED: MPPI WILL NOT DRIVE THIS ROBOT

  It loads cleanly and commands 0.0034 m/s; its own optimal trajectory
  advances 0.4 mm per step; goal ABORTED after 154 s and 1.1 m of
  recoveries. Everything it consumes was verified good on the same runs -
  plan, transformed plan, free local costmap, footprint, all 8 critics
  loaded with the configured weights, every parameter reading back
  correctly - and the same stack drives 63.6 m under the survey node and
  reaches this goal in 20.5 s under RegulatedPurePursuit.
  consider_footprint and regenerate_noises were bisected out.

  Phase 1 therefore ships with RegulatedPurePursuit. THIS IS A DEPARTURE
  FROM docs/PLAN.md SECTION 1 AND NEEDS A DECISION. The MPPI block is
  preserved verbatim as FollowPath_mppi_deferred; reverting is a rename of
  two keys. Nothing else in the stack assumes which controller is loaded.

Verification: 9 packages build, 39 tests pass, flake8 + black clean.

File: src/amr_description/urdf/amr.urdf.xacro (robot description, xacro)
@@ -210,4 +210,31 @@
   </xacro:macro>
   <xacro:caster side="front" reflect="1"/>
+  <!-- Sensor mast. Visual only: the chassis already provides collision, and a mast
+       with collision geometry would be one more thing for the LiDAR to see. It exists
+       because lidar_height now puts the scan plane ABOVE the chassis rather than
+       inside it - see fleet.yaml - and a sensor floating in mid-air above the body
+       reads as a modelling mistake in a demo even when the physics is right. -->
+  <xacro:property name="mast_top" value="${lidar_height - wheel_radius}"/>
+  <xacro:property name="mast_bottom" value="${base_height}"/>
+  <link name="${prefix}mast">
+    <visual>
+      <origin xyz="0 0 ${(mast_top + mast_bottom) / 2.0}" rpy="0 0 0"/>
+      <geometry>
+        <box size="0.06 0.06 ${mast_top - mast_bottom}"/>
+      </geometry>
+      <material name="amr_mast">
+        <color rgba="0.3 0.3 0.32 1.0"/>
+      </material>
+    </visual>
+    <inertial>
+      <mass value="0.05"/>
+      <inertia ixx="1e-5" ixy="0.0" ixz="0.0" iyy="1e-5" iyz="0.0" izz="1e-5"/>
+    </inertial>
+  </link>
+  <joint name="${prefix}mast_joint" type="fixed">
+    <parent link="${prefix}base_link"/>
+    <child link="${prefix}mast"/>
+    <origin xyz="${body_x + base_length / 2.0 - 0.06} 0 0" rpy="0 0 0"/>
+  </joint>
   <!-- 2D LiDAR. Height above ground is the tunable that smoke test 2 informs. -->
   <link name="${prefix}laser">

Commit message: feat(phase2): SensorBSP validators + PitchGate, and the SafetyGate override
SensorBSP relays every sensor through a plausibility check and republishes on
validated/* topics, preserving the original header stamp (rule 4). Nav2 and
slam_toolbox now consume validated topics only (rule 8); the instruments that
measure the BSP subscribe to both sides by design and say so.

PitchGate truncates ground returns per beam at margin * h / (sin|pitch| cos az),
using the buffered IMU sample NEAREST each scan's own stamp rather than the
latest received. Truncation is floored by d_safe(v_max) + footprint + margin, so
it can never delete an obstacle the gate would have had to stop for; the
interlock is pinned by tests rather than by a launch file being correct.

SafetyGate is a serial, fail-closed gate and the last link before cmd_vel
(rule 1), sized by d_safe = k*v^2 + d_min on MEASURED odometry velocity (rule 3)
with k derived from fleet.yaml mass, payload and decel limit. It suppresses
Nav2's progress checker while it holds the robot (rule 2) and restores it only
after real motion. C++ because it is in the command path; the sizing arithmetic
is Python so pytest owns it. No robot name appears in either (rule 5).

Evidence, all in results/:
  PitchGate      903 stamp-exact raw/validated pairs, 0 restamped, 0 ns drift;
                 120 beams cut at 8.001 deg, closest removed 2.769 m against a
                 2.263 m gate; 0 cut uphill, inside gate, or inside the envelope
  IMU injection  500 samples at 50 rad/s rejected, 0 reached validated/imu,
                 3194 healthy samples accepted around them
  Safety halt    goal SUCCEEDED, 3 halts, 0 commands leaked while latched,
                 sensor stamp -> zero published 8.46 / 11.00 / 12.00 ms
  Stopping sweep four speeds, k_model 1.875 vs k_measured 1.021 s^2/m, both
                 quoted because the simulator brakes kinematically
  Fail-closed    SIGKILL mid-motion: 0.196 m to rest with the plant watchdog,
                 still rolling at 0.350 m/s after 3.500 m without it

Two corrections this phase, both to conclusions rather than to code. The earlier
"a second rendering sensor stalls the drive" finding is retracted: re-measured on
a clean process table the camera makes no difference (0.3500 m/s either way), and
the real cause was leaked drive_watchdog processes from previous launches
contending on the plant command topic. And the recovery-suppression A/B is
reported as NOT having exercised the mechanism - both arms show zero recoveries
during a halt because no halt approached the 10 s allowance. The parameter
read-back shows the mechanism operates; necessity is left unproven and flagged.

File: src/amr_description/urdf/amr.urdf.xacro (robot description, xacro)
@@ -43,4 +43,34 @@
   <xacro:arg name="lidar_update_rate" default="10.0"/>
   <xacro:arg name="imu_update_rate" default="100.0"/>
+  <!-- ==== Forward camera - PRESENT, DEFAULTED OFF, AND IT DOES NOT COST MOTION ====
+       The assignment's evaluation table asks for a camera validator, and a validator
+       with no camera behind it is dead code, so a deliberately tiny 160x120 sensor at
+       10 Hz gives CameraValidator live stamps, resolution and encoding to check.
+       A CORRECTED FINDING. An earlier session recorded that enabling this camera
+       stalled the drive - commanded 0.35 m/s, achieved 0.00017 m/s - and defaulted it
+       off for that reason. That attribution was WRONG. The stall was caused by
+       drive_watchdog processes leaked from earlier launches, still subscribed to
+       /amrN/cmd_vel and republishing onto /amrN/cmd_vel_plant; the contention starved
+       the graph until the gate's own command-timeout fired and interleaved zeros into
+       the command stream, so DiffDrive's acceleration limit never integrated. The
+       camera happened to be the variable under test at the time.
+       Re-measured on a verified-clean process table, one variable, everything else
+       identical (results/phase2_camera_motion_{on,off}.md):
+           camera ENABLED  : commanded 0.35 m/s, peak measured 0.3500 m/s, 13.53 m
+           camera DISABLED : commanded 0.35 m/s, peak measured 0.3500 m/s, 13.86 m
+       Identical peak speed. The remaining 2 % of distance is where the fixed sim-time
+       window happened to close, not a motion deficit.
+       So why still default OFF? Because the camera has no downstream consumer in this
+       project - nothing plans, localises or avoids with it - and every extra rendering
+       sensor is load this 6 GB GPU does not need to carry on a run that does not use
+       it. That is a cost decision, not a defect workaround, and it is reversible by
+       flipping this one argument.
+       camera_enabled is a per-RUN switch, not a per-robot property, so it is absent
+       from fleet.yaml. bsp.launch.py's camera_enabled argument must be kept in step
+       with this one, or the BSP subscribes to a topic nobody publishes. -->
+  <xacro:arg name="camera_enabled" default="false"/>
+  <xacro:arg name="camera_width" default="160"/>
+  <xacro:arg name="camera_height" default="120"/>
+  <xacro:arg name="camera_update_rate" default="10.0"/>
   <!-- ==== Kinodynamic limits (also fed to nav2_velocity_smoother in later phases,
            so simulation and planning read the SAME numbers) ==== -->
@@ -268,4 +298,18 @@
     <origin xyz="${body_x} 0 ${base_height / 2.0}" rpy="0 0 0"/>
   </joint>
+  <!-- Forward camera, on the front face of the chassis looking down the +x axis. -->
+  <xacro:if value="$(arg camera_enabled)">
+    <link name="${prefix}camera_link">
+      <inertial>
+        <mass value="0.02"/>
+        <inertia ixx="1e-6" ixy="0.0" ixz="0.0" iyy="1e-6" iyz="0.0" izz="1e-6"/>
+      </inertial>
+    </link>
+    <joint name="${prefix}camera_joint" type="fixed">
+      <parent link="${prefix}base_link"/>
+      <child link="${prefix}camera_link"/>
+      <origin xyz="${body_x + base_length / 2.0} 0 ${base_height / 2.0}" rpy="0 0 0"/>
+    </joint>
+  </xacro:if>
   <!-- Gazebo sensors, materials and the differential drive system. -->
   <!-- Relative include: resolves both in-source and from the installed share/

File: src/amr_description/urdf/amr_gazebo.xacro (robot description, xacro)
@@ -83,4 +83,28 @@
     </sensor>
   </gazebo>
+  <!-- ==================== Forward camera ==================== -->
+  <xacro:if value="$(arg camera_enabled)">
+    <gazebo reference="${prefix}camera_link">
+      <sensor name="camera" type="camera">
+        <topic>${name}/camera/image_raw</topic>
+        <update_rate>$(arg camera_update_rate)</update_rate>
+        <always_on>1</always_on>
+        <camera>
+          <horizontal_fov>1.047</horizontal_fov>
+          <image>
+            <width>$(arg camera_width)</width>
+            <height>$(arg camera_height)</height>
+            <!-- R8G8B8 bridges to the ROS encoding "rgb8", which is what
+                 amr_bsp.validators.CAMERA_ENCODINGS accepts. -->
+            <format>R8G8B8</format>
+          </image>
+          <clip>
+            <near>0.1</near>
+            <far>15.0</far>
+          </clip>
+        </camera>
+      </sensor>
+    </gazebo>
+  </xacro:if>
   <!-- ==================== Systems ==================== -->
   <gazebo>
@@ -100,5 +124,15 @@
       <max_angular_acceleration>$(arg max_accel_theta)</max_angular_acceleration>
       <min_angular_acceleration>${-1.0 * $(arg max_accel_theta)}</min_angular_acceleration>
-      <topic>${name}/cmd_vel</topic>
+      <!-- cmd_vel_plant, NOT cmd_vel. /amrN/cmd_vel is what SafetyGate publishes and
+           is the robot's command topic; this is the wheel controller's input, one hop
+           further in, behind amr_gazebo's drive_watchdog.
+           The watchdog exists because gz-sim 8.11.0's DiffDrive has no command
+           timeout - verified against the plugin binary, whose only cmd-related string
+           is the topic name. Without it, a SIGKILLed SafetyGate leaves the plant
+           rolling on the last velocity it latched, and "if the node dies, nothing
+           moves" (docs/ENGINEERING_NOTES.md rule 1) would be a claim the simulator cannot honour.
+           Real motor controllers stop when their command stream stops; the watchdog
+           models exactly that and belongs to the plant, not to the nav stack. -->
+      <topic>${name}/cmd_vel_plant</topic>
       <odom_topic>${name}/odom</odom_topic>
       <tf_topic>${name}/pose</tf_topic>
