Commit message: feat: cooperative mapping demo in RViz, and the launch bug that hid it
RViz came up blank on "Frame [map] does not exist" for every fleet demo. Two
causes, both fixed.

The saved config was never loaded. Launch configurations are inherited by
included launch descriptions, and DeclareLaunchArgument only supplies a default
for a name that is not already set - so phase3's own `rviz_config`, declared
with an empty default to avoid restating the path, leaked into fleet_nav and
won over fleet_nav's real default. RViz was started as `-d ""` and silently
fell back to its stock config. fleet_nav now resolves an empty value to
DEFAULT_RVIZ_CONFIG, so the path stays written down once and an empty value
means "the default" from any caller.

And `map` is not a frame this system publishes: every SLAM frame is namespaced
amrN/map and the shared root is fleet_map, which FleetMapNode publishes at
t=16s. Verified at runtime rather than assumed - tf2_echo fleet_map
amr1/base_link resolves and tracks the moving robot.

rviz/fleet_mapping.rviz: /fleet_map, both robot models (blue amr1, amber amr2
via body_color in fleet.yaml, because RobotModel has no colour property), both
scans, both plans, key TF frames only, warehouse top-down. Own-maps, global
costmaps, predicted trajectories and local costmaps ship as off-by-default
toggles so one config serves the mapping and MAPF demos.

fleet_survey.launch.py is the cooperative mapping demo: the fleet stack with
Nav2 left out and a scripted drive per robot, both on the same circuit half a
lap apart, so /fleet_map fills in from both ends of the aisle at once. GUI and
RViz on by default - it is the one launch built for the camera.

rviz:=true now also on phase6_conflict and phase7_yield, so every two-robot
demo can start RViz inside the launch rather than beside it.

Dynamic obstacles were implemented and working but switched off in the demo the
runbook told you to record: phase3_fleet_goals defaults with_actors:=false.
Defaults left alone - flipping one would change the configuration its committed
artifact was measured in - and documented per launch instead, with the
recording command passing with_actors:=true tag:=demo. Verified: all three
pedestrians render and both goals still SUCCEEDED.

DEMO_RUNBOOK rewritten. Every command checked against the launch file it names;
all the pre-existing ones were valid. Each demo now carries purpose, terminals,
startup sequence, duration, what to point out, expected result, failure modes
and how to stop cleanly, plus a dynamic-obstacle table.

Submission cleanup: PLAN.md and SESSION_LOG.md are properly removed rather than
emptied, and the nine source files plus five README passages that cited them
repointed at the README section or results/ artifact holding the same fact.
ENGINEERING_NOTES kept - the code cites its rules by number. videos/ added for
the screenshare, which is delivered separately and git-ignored along with
*.mp4/*.mkv/*.webm, less the four short evidence clips in media/.

README: mapping demo and RViz instructions, a dynamic-obstacles section, and
two new limitations stated plainly - that most measurement runs were made with
pedestrians off, and that the survey demo's own numbers are not the committed
selective-mapping evidence.

Build 9 packages 0 errors, 241 tests pass, flake8 and black clean.

File: src/amr_description/urdf/amr.urdf.xacro (robot description, xacro)
@@ -73,4 +73,11 @@
   <xacro:arg name="camera_height" default="120"/>
   <xacro:arg name="camera_update_rate" default="10.0"/>
+  <!-- Chassis colour, "r g b a" in 0..1. Visual only - it reaches the RViz
+       RobotModel display and the Gazebo visual, and nothing else reads it. It
+       exists because rviz_default_plugins/RobotModel has no colour override
+       property: two robots from one xacro are indistinguishable on screen unless
+       the difference is in the description. Default is the original body colour,
+       so a fleet entry that omits it renders exactly as before. -->
+  <xacro:arg name="body_color" default="0.25 0.35 0.55 1.0"/>
   <!-- ==== Kinodynamic limits (also fed to nav2_velocity_smoother in later phases,
            so simulation and planning read the SAME numbers) ==== -->
@@ -92,4 +99,5 @@
   <xacro:property name="base_height" value="$(arg base_height)"/>
   <xacro:property name="lidar_height" value="$(arg lidar_height)"/>
+  <xacro:property name="body_color" value="$(arg body_color)"/>
   <!-- Total mass is what the physics engine sees; payload scaling elsewhere in the
        stack (SafetyGate's k, PayloadJerkAdapter's limits) keys off payload_kg. -->
@@ -141,6 +149,6 @@
         <box size="${base_length} ${base_width} ${base_height}"/>
       </geometry>
-      <material name="amr_body">
-        <color rgba="0.25 0.35 0.55 1.0"/>
+      <material name="${name}_body">
+        <color rgba="${body_color}"/>
       </material>
     </visual>
